Commit message: Update files and docs to align with single computer setup.

File: ad_r1m_perception_cuvslam/urdf/single_realsense_calibration.urdf.xacro (robot description, xacro)
@@ -1,7 +1,7 @@
 <?xml version="1.0"?>
 <robot name="adrd_demo_ros2">
-  <link name="ad_r1m_0/base_link" />
+  <link name="base_link" />
   <joint name="camera1" type="fixed">
-    <parent link="ad_r1m_0/base_link"/>
+    <parent link="base_link"/>
     <child link="camera1_link"/>
     <origin xyz="0.335 0.0 0.0" rpy="0 0 0"/>
