Commit message: Modify package's information.

File: ad_r1m_perception_cuvslam/urdf/realsense_calibration.urdf.xacro (robot description, xacro)
@@ -1,3 +1,3 @@
-<?xml version="1.0">
+<?xml version="1.0"?>
 <robot name="4_realsenses">
   <link name="base_link"/>

File: ad_r1m_perception_cuvslam/urdf/single_realsense_calibration.urdf.xacro (robot description, xacro)
@@ -1,3 +1,3 @@
-<?xml version="1.0">
+<?xml version="1.0"?>
 <robot name="adrd_demo_ros2">
   <link name="ad_r1m_0/base_link" />
@@ -8,9 +8,3 @@
   </joint>
   <link name="camera1_link"/>
-  <link name="camera_imu_optical_frame"/>
-  <joint name="camera1_to_imu" type="fixed">
-    <parent link="camera1_link"/>
-    <child link="camera_imu_optical_frame"/>
-    <origin xyz="0 0 0" rpy="0 0 0"/>
-  </joint>
 </robot>
