Commit message: Align the configurations with custom build.

File: ad_r1m_description/urdf/ad_r1m_base.urdf.xacro (robot description, xacro)
@@ -6,7 +6,7 @@
 <xacro:include filename="_imu_adis16470.xacro" />
 <xacro:macro name="ad_r1m_base" params="prefix use_sim:=false">
-    <xacro:property name="chassis_length" value="0.59"/>
-    <xacro:property name="chassis_width" value="0.36"/>
-    <xacro:property name="chassis_height" value="0.12"/>
+    <xacro:property name="chassis_length" value="0.68"/> <!-- CHANGED -->
+    <xacro:property name="chassis_width" value="0.34"/>
+    <xacro:property name="chassis_height" value="0.15"/> <!-- CHANGED -->
     <xacro:property name="base_width" value="0.22"/>
     <xacro:property name="wheel_separation" value="0.29"/>
@@ -15,5 +15,5 @@
     <xacro:property name="chassis_mass" value="1.0"/>
     <xacro:property name="wheel_radius" value="0.05"/>
-    <xacro:property name="wheel_width" value="0.025"/>
+    <xacro:property name="wheel_width" value="0.03"/> <!-- CHANGED -->
     <xacro:property name="wheel_mass" value="0.5"/> <!-- SLIP_FIX was 0.05 -->
     <xacro:property name="caster_wheel_radius" value="0.025"/>
@@ -35,5 +35,5 @@
     <!-- HARDWARE MODULES -->
     <xacro:imu_adis16470 prefix="${prefix}" parent="${prefix}base_link">
-        <origin xyz="0.180 0 ${wheel_radius}" rpy="${pi} 0 ${-pi/2}"/>
+        <origin xyz="-0.120 0.04 ${wheel_radius}" rpy="0 0 ${-pi}"/>
     </xacro:imu_adis16470>
     <xacro:tof_adtf3175d prefix="${prefix}" parent="${prefix}base_link" use_sim="${use_sim}">
